File: kicad-10outputs/10outputs.kicad_sch (KiCad schematic)
At the start: 29 parts, among them J1 Conn_01x03_Male, J2 Conn_01x06_Male, J3 Conn_01x06_Male, J4 Conn_01x02_Male, J5 Conn_01x01_Male, J6 Conn_01x01_Male, Q1 BSP75N, Q10 BSP75N, Q2 BSP75N, Q3 BSP75N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

Commit message: feat: add 5 outputs
Parts:
- R1: value 3k -> 1k
- R2: renamed from 1k1; value R -> R2
Changed lines of the file:
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@@
     (in_bom yes) (on_board yes) (fields_autoplaced)
     (property "Reference" "R1" (id 0) (at 109.22 76.2 90))
-    (property "Value" "3k" (id 1) (at 109.22 78.74 90))
+    (property "Value" "1k" (id 1) (at 109.22 78.74 90))
     (property "Footprint" "Resistor_SMD:R_0805_2012Metric_Pad1.20x1.40mm_HandSolder" (id 2) (at 109.22 84.328 90)
       (effects (font (size 1.27 1.27)) hide)
@@
   (symbol (lib_id "Device:R") (at 83.82 82.55 90) (unit 1)
     (in_bom yes) (on_board yes) (fields_autoplaced)
-    (property "Reference" "1k1" (id 0) (at 83.82 76.2 90))
-    (property "Value" "R" (id 1) (at 83.82 78.74 90))
+    (property "Reference" "R2" (id 0) (at 83.82 76.2 90))
+    (property "Value" "R2" (id 1) (at 83.82 78.74 90))
     (property "Footprint" "Resistor_SMD:R_0805_2012Metric_Pad1.20x1.40mm_HandSolder" (id 2) (at 83.82 84.328 90)
       (effects (font (size 1.27 1.27)) hide)
@@
       (reference "#PWR0124") (unit 1) (value "+3.3V") (footprint "")
     )
-    (path "/e3c4a5c0-6a22-4316-8c8d-e2edf7314b52"
-      (reference "1k1") (unit 1) (value "R") (footprint "Resistor_SMD:R_0805_2012Metric_Pad1.20x1.40mm_HandSolder")
-    )
     (path "/308b40b6-6a8d-4fcf-8b19-b462d3a7d546"
       (reference "10nF1") (unit 1) (value "C") (footprint "Capacitor_SMD:C_0805_2012Metric_Pad1.18x1.45mm_HandSolder")
@@
     )
     (path "/d192c122-2689-4f00-8477-01527b6defde"
-      (reference "R1") (unit 1) (value "3k") (footprint "Resistor_SMD:R_0805_2012Metric_Pad1.20x1.40mm_HandSolder")
+      (reference "R1") (unit 1) (value "1k") (footprint "Resistor_SMD:R_0805_2012Metric_Pad1.20x1.40mm_HandSolder")
+    )
+    (path "/e3c4a5c0-6a22-4316-8c8d-e2edf7314b52"
+      (reference "R2") (unit 1) (value "R2") (footprint "Resistor_SMD:R_0805_2012Metric_Pad1.20x1.40mm_HandSolder")
     )
     (path "/c8bc6c7a-10f0-42f1-abdd-c4ff03a9c06a"
