File: kicad-9outputs/9outputs.kicad_sch (KiCad schematic)
At the start: 20 parts, among them J1 Screw_Terminal_01x04, J11 Screw_Terminal_01x02, J2 Screw_Terminal_01x04, J3 Screw_Terminal_01x04, J4 Screw_Terminal_01x03, Q1 BSP75N, Q2 BSP75N, Q3 BSP75N, Q4 BSP75N, Q5 BSP75N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

Commit message: feat: add 5 outputs
Parts:
- added R1, R2, R3: R, Resistor_SMD:R_1206_3216Metric_Pad1.30x1.75mm_HandSolder, symbol Device:R
- 1111: renamed from 111; footprint kpjx:KPJX4SS -> custom2:KPJX4SS
Connections:
- net +3.3V: now also R2.1
- net GND: now also R1.2, R3.2
- net IN1: now also R1.1
- net IN2: now also R2.2, R3.1
